File: hardware/pcb/switch_matrix.kicad_sch (KiCad schematic)
At the start: 32 parts, among them SW1 SW_Push, SW10 SW_Push, SW11 SW_Push, SW12 SW_Push, SW13 SW_Push, SW14 SW_Push, SW15 SW_Push, SW16 SW_Push, SW2 SW_Push, SW3 SW_Push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

Commit message: Update PCB and production files to revision 2
Parts:
- SW1, SW10, SW11, SW12, SW13, SW14, SW15, SW16, SW2, SW3, SW4, SW5, SW6, SW7, SW8, SW9: footprint Keyboard switches:SW_Gateron_LowProfile_THT -> key-switches:SW_Gateron_LowProfile_THT
Changed lines of the file:
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@@
       (effects (font (size 1.27 1.27)))
     )
-    (property "Footprint" "Keyboard switches:SW_Gateron_LowProfile_THT" (at 120.65 99.06 0)
+    (property "Footprint" "key-switches:SW_Gateron_LowProfile_THT" (at 120.65 99.06 0)
       (effects (font (size 1.27 1.27)) hide)
     )
@@
       (effects (font (size 1.27 1.27)))
     )
-    (property "Footprint" "Keyboard switches:SW_Gateron_LowProfile_THT" (at 120.65 52.07 0)
+    (property "Footprint" "key-switches:SW_Gateron_LowProfile_THT" (at 120.65 52.07 0)
       (effects (font (size 1.27 1.27)) hide)
     )
@@
       (effects (font (size 1.27 1.27)))
     )
-    (property "Footprint" "Keyboard switches:SW_Gateron_LowProfile_THT" (at 163.83 99.06 0)
+    (property "Footprint" "key-switches:SW_Gateron_LowProfile_THT" (at 163.83 99.06 0)
       (effects (font (size 1.27 1.27)) hide)
     )
@@
       (effects (font (size 1.27 1.27)))
     )
-    (property "Footprint" "Keyboard switches:SW_Gateron_LowProfile_THT" (at 186.69 99.06 0)
+    (property "Footprint" "key-switches:SW_Gateron_LowProfile_THT" (at 186.69 99.06 0)
       (effects (font (size 1.27 1.27)) hide)
     )
@@
       (effects (font (size 1.27 1.27)))
     )
-    (property "Footprint" "Keyboard switches:SW_Gateron_LowProfile_THT" (at 163.83 74.93 0)
+    (property "Footprint" "key-switches:SW_Gateron_LowProfile_THT" (at 163.83 74.93 0)
       (effects (font (size 1.27 1.27)) hide)
     )
@@
       (effects (font (size 1.27 1.27)))
     )
-    (property "Footprint" "Keyboard switches:SW_Gateron_LowProfile_THT" (at 99.06 99.06 0)
+    (property "Footprint" "key-switches:SW_Gateron_LowProfile_THT" (at 99.06 99.06 0)
       (effects (font (size 1.27 1.27)) hide)
     )
@@
       (effects (font (size 1.27 1.27)))
     )
-    (property "Footprint" "Keyboard switches:SW_Gateron_LowProfile_THT" (at 99.06 52.07 0)
+    (property "Footprint" "key-switches:SW_Gateron_LowProfile_THT" (at 99.06 52.07 0)
       (effects (font (size 1.27 1.27)) hide)
     )
@@
       (effects (font (size 1.27 1.27)))
     )
-    (property "Footprint" "Keyboard switches:SW_Gateron_LowProfile_THT" (at 186.69 123.19 0)
+    (property "Footprint" "key-switches:SW_Gateron_LowProfile_THT" (at 186.69 123.19 0)
       (effects (font (size 1.27 1.27)) hide)
     )
@@
       (effects (font (size 1.27 1.27)))
     )
-    (property "Footprint" "Keyboard switches:SW_Gateron_LowProfile_THT" (at 120.65 74.93 0)
+    (property "Footprint" "key-switches:SW_Gateron_LowProfile_THT" (at 120.65 74.93 0)
       (effects (font (size 1.27 1.27)) hide)
     )
@@
       (effects (font (size 1.27 1.27)))
     )
-    (property "Footprint" "Keyboard switches:SW_Gateron_LowProfile_THT" (at 142.24 74.93 0)
+    (property "Footprint" "key-switches:SW_Gateron_LowProfile_THT" (at 142.24 74.93 0)
       (effects (font (size 1.27 1.27)) hide)
     )
@@
       (effects (font (size 1.27 1.27)))
     )
-    (property "Footprint" "Keyboard switches:SW_Gateron_LowProfile_THT" (at 142.24 99.06 0)
+    (property "Footprint" "key-switches:SW_Gateron_LowProfile_THT" (at 142.24 99.06 0)
       (effects (font (size 1.27 1.27)) hide)
     )
@@
       (effects (font (size 1.27 1.27)))
     )
-    (property "Footprint" "Keyboard switches:SW_Gateron_LowProfile_THT" (at 142.24 123.19 0)
+    (property "Footprint" "key-switches:SW_Gateron_LowProfile_THT" (at 142.24 123.19 0)
       (effects (font (size 1.27 1.27)) hide)
     )
@@
       (effects (font (size 1.27 1.27)))
     )
-    (property "Footprint" "Keyboard switches:SW_Gateron_LowProfile_THT" (at 142.24 52.07 0)
+    (property "Footprint" "key-switches:SW_Gateron_LowProfile_THT" (at 142.24 52.07 0)
       (effects (font (size 1.27 1.27)) hide)
     )
@@
       (effects (font (size 1.27 1.27)))
     )
-    (property "Footprint" "Keyboard switches:SW_Gateron_LowProfile_THT" (at 163.83 52.07 0)
+    (property "Footprint" "key-switches:SW_Gateron_LowProfile_THT" (at 163.83 52.07 0)
       (effects (font (size 1.27 1.27)) hide)
     )
@@
       (effects (font (size 1.27 1.27)))
     )
-    (property "Footprint" "Keyboard switches:SW_Gateron_LowProfile_THT" (at 186.69 52.07 0)
+    (property "Footprint" "key-switches:SW_Gateron_LowProfile_THT" (at 186.69 52.07 0)
       (effects (font (size 1.27 1.27)) hide)
     )
@@
       (effects (font (size 1.27 1.27)))
     )
-    (property "Footprint" "Keyboard switches:SW_Gateron_LowProfile_THT" (at 186.69 74.93 0)
-      (effects (font (size 1.27 1.27)) hide)
-    )
+    (property "Footprint" "key-switches:SW_Gateron_LowProfile_THT" (at 186.69 74.93 0)
+      (effects (font (size 1.27 1.27)) hide)
+    )

Commit message: Version 2 sent to production
Parts:
- SW1, SW10, SW11, SW12, SW13, SW14, SW15, SW16, SW2, SW3, SW4, SW5, SW6, SW7, SW8, SW9: now not fitted
Changed lines of the file:
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@@
 		(in_bom yes)
 		(on_board yes)
-		(dnp no)
+		(dnp yes)
 		(fields_autoplaced yes)
 		(property "Reference" "SW11"
@@
 		(in_bom yes)
 		(on_board yes)
-		(dnp no)
+		(dnp yes)
 		(fields_autoplaced yes)
 		(property "Reference" "SW2"
@@
 		(in_bom yes)
 		(on_board yes)
-		(dnp no)
+		(dnp yes)
 		(fields_autoplaced yes)
 		(property "Reference" "SW13"
@@
 		(in_bom yes)
 		(on_board yes)
-		(dnp no)
+		(dnp yes)
 		(fields_autoplaced yes)
 		(property "Reference" "SW14"
@@
 		(in_bom yes)
 		(on_board yes)
-		(dnp no)
+		(dnp yes)
 		(fields_autoplaced yes)
 		(property "Reference" "SW8"
@@
 		(in_bom yes)
 		(on_board yes)
-		(dnp no)
+		(dnp yes)
 		(fields_autoplaced yes)
 		(property "Reference" "SW10"
@@
 		(in_bom yes)
 		(on_board yes)
-		(dnp no)
+		(dnp yes)
 		(fields_autoplaced yes)
 		(property "Reference" "SW1"
@@
 		(in_bom yes)
 		(on_board yes)
-		(dnp no)
+		(dnp yes)
 		(fields_autoplaced yes)
 		(property "Reference" "SW16"
@@
 		(in_bom yes)
 		(on_board yes)
-		(dnp no)
+		(dnp yes)
 		(fields_autoplaced yes)
 		(property "Reference" "SW6"
@@
 		(in_bom yes)
 		(on_board yes)
-		(dnp no)
+		(dnp yes)
 		(fields_autoplaced yes)
 		(property "Reference" "SW7"
@@
 		(in_bom yes)
 		(on_board yes)
-		(dnp no)
+		(dnp yes)
 		(fields_autoplaced yes)
 		(property "Reference" "SW12"
@@
 		(in_bom yes)
 		(on_board yes)
-		(dnp no)
+		(dnp yes)
 		(fields_autoplaced yes)
 		(property "Reference" "SW15"
@@
 		(in_bom yes)
 		(on_board yes)
-		(dnp no)
+		(dnp yes)
 		(fields_autoplaced yes)
 		(property "Reference" "SW3"
@@
 		(in_bom no)
 		(on_board yes)
-		(dnp no)
+		(dnp yes)
 		(fields_autoplaced yes)
 		(property "Reference" "SW4"
@@
 		(in_bom yes)
 		(on_board yes)
-		(dnp no)
+		(dnp yes)
 		(fields_autoplaced yes)
 		(property "Reference" "SW5"
@@
 		(in_bom yes)
 		(on_board yes)
-		(dnp no)
+		(dnp yes)
 		(fields_autoplaced yes)
 		(property "Reference" "SW9"

Commit message: V1.5
Other:
- note added: "All swiches are Do Not Place. They must be populated by hand."
- title: (none) -> Mathboard 
Changed lines of the file:
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@@
 	(generator_version "8.0")
 	(paper "A4")
+	(title_block
+		(title "Mathboard ")
+		(date "2025-01-16")
+		(rev "1.5")
+	)
 	(junction
 		(at 195.58 80.01)
@@
 		)
 	)
+	(text "All swiches are Do Not Place. They must be populated by hand."
+		(exclude_from_sim no)
+		(at 112.522 29.718 0)
+		(effects
+			(font
+				(size 1.27 1.27)
+			)
+		)
+	)
