File: hardware/pcb/switch_matrix.kicad_sch (KiCad schematic)
At the start: 38 parts, among them SW1 SW_socket, SW10 SW_socket, SW11 SW_socket, SW12 SW_socket, SW13 SW_socket, SW14 SW_socket, SW15 SW_socket, SW16 SW_socket, SW2 SW_socket, SW3 SW_socket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

Commit message: Remove old Mathboard kicad project
Parts:
- SW1, SW10, SW11, SW12, SW13, SW14, SW15, SW16, SW2, SW3, SW4, SW5, SW6, SW7, SW8, SW9: footprint mathboard:SW_Gateron_LowProfile_THT_hotswap -> mathpad:SW_Gateron_LowProfile_THT_hotswap; JLCPCB BOM 0 -> (none)
Other:
- company: (none) -> Summacogni OÜ
- title: (none) -> Mathpad
- moved on the sheet: C22, C24, C25, C26, C27, C9
