File: hardware/pcb/kicad/Mathpad.kicad_sch (KiCad schematic)
At the start: 21 parts, among them J1 TYPE-C sinking plate, SW17 MSK13C02, U2 SK6812-MINI-E, U3 USBLC6-2P6, U4 XC6206P332MR-G

Commit message: Reformatting, removing old files, add better documentation about licenses
Other:
- title: Mathpad -> Mathpad PCB
Changed lines of the file:
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@@
 	(paper "A4")
 	(title_block
-		(title "Mathpad")
-		(date "2025-04-05")
+		(title "Mathpad PCB")
+		(date "2025-04-07")
 		(rev "1.6")
 		(company "Summacogni OÜ")

Commit message: Minor modifications to the pcb
Parts:
- removed D17: D_Zener, mathpad:DFN1006-2L, symbol Device:D_Zener
- removed D19: DSL14, Diode_SMD:D_SOD-123, symbol Device:D_Schottky
- U3: JLCPCB_CORRECTION 0; 0; 270 -> (none)
Connections:
- net +5V: now also F1.2, U3.5 (VBUS)
Other:
- moved on the sheet: F1, U3

Commit message: ChangePCB thickness to 1mm
Parts:
- J1: footprint mathpad:USB_C_Receptacle_XYECONN TYPE-C-F02C-1BBWC1.6 -> mathpad:USB_C_Receptacle_GT-USB-7014B01; JLCPCB Part # (none) -> C963372; LCSC C20883026 -> (none); MPN  TYPE-C-F02C-1BBWC1.6 -> 7014B
Changed lines of the file:
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@@
 		(title "Mathpad PCB")
 		(date "2025-04-07")
-		(rev "1.6")
+		(rev "1.7")
 		(company "Summacogni OÜ")
 	)
@@
 			)
 		)
-		(property "Footprint" "mathpad:USB_C_Receptacle_XYECONN TYPE-C-F02C-1BBWC1.6"
+		(property "Footprint" "mathpad:USB_C_Receptacle_GT-USB-7014B01"
 			(at 52.07 120.65 0)
 			(effects
@@
 			)
 		)
-		(property "Datasheet" "https://wmsc.lcsc.com/wmsc/upload/file/pdf/v2/lcsc/2403011808_XYECONN-TYPE-C-F02C-1BBWC1-6_C20883026.pdf"
+		(property "Datasheet" "https://www.lcsc.com/datasheet/lcsc_datasheet_2411221125_G-Switch-GT-USB-7014B01_C19188078.pdf"
 			(at 52.07 120.65 0)
 			(effects
@@
 			)
 		)
-		(property "MPN " "TYPE-C-F02C-1BBWC1.6"
+		(property "MPN " "7014B"
 			(at 48.26 120.65 0)
 			(effects
@@
 			)
 		)
-		(property "LCSC" "C20883026"
+		(property "LCSC" ""
 			(at 48.26 120.65 0)
 			(effects
@@
 			)
 		)
-		(property "JLCPCB Part #" ""
+		(property "JLCPCB Part #" "C963372"
 			(at 48.26 120.65 0)
 			(effects

Commit message: Add MPN and purchase links to all components
Parts:
- C1: value 100n -> 100nF X7R ±10% 16V; MPN  100nF 10% 10V 0402 -> CL05B104KO5NNNC; Purchase link (none) -> https://lcsc.com/product-detail/Multilayer-Ceramic-Capacito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
- C20, C21: value 4.7u -> 4.7uF X5R ±10% 10V; MPN  4.7uF 20% 10V 0402 -> CL10A475KP8NNNC; Purchase link (none) -> https://lcsc.com/product-detail/Multilayer-Ceramic-Capacito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
- D18: MPN  (none) -> A-SP192SGHC-C01-3C; Purchase link (none) -> https://lcsc.com/product-detail/LED-Indication-Discrete_Ami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
- F1: Purchase link (none) -> https://lcsc.com/product-detail/Resettable-Fuses_BHFUSE-BSM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
- J1: JLCPCB Part # C963372 -> (none); LCSC (none) -> C963372; MPN  7014B -> GT-USB-7014B; Purchase link (none) -> https://lcsc.com/product-detail/USB-Connectors_G-Switch-GT-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
- R10, R15: MPN  10k 1% 0402 -> 0402WGF1002TCE; Purchase link (none) -> https://lcsc.com/product-detail/Chip-Resistor-Surface-Mount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
- R18: value 1k -> 1k 1%; MPN  1k 1% 0402 -> 0402WGF1001TCE; Purchase link (none) -> https://lcsc.com/product-detail/Chip-Resistor-Surface-Mount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
- R19, R7, R8: value 5.1k -> 5.1k 1%; MPN  5.1k 1% 0402 -> 0402WGF5101TCE; Purchase link (none) -> https://lcsc.com/product-detail/Chip-Resistor-Surface-Mount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
- SW17: value MSK13C02 -> SP3T; MPN  (none) -> MSK13C02; Purchase link (none) -> https://lcsc.com/product-detail/Slide-Switches_SHOU-HAN-MSK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
- U2: value SK6812-MINI-E -> SK6812MINI-E; MPN  (none) -> SK6812MINI-E; Purchase link (none) -> https://lcsc.com/product-detail/RGB-LEDs-Built-in-IC_OPSCO-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
- U3: Purchase link (none) -> https://lcsc.com/product-detail/ESD-and-Surge-Protection-TV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
- U4: value XC6206P332MR-G -> 3.3V 200mA LDO; MPN  (none) -> XC6206P332MR-G; Purchase link (none) -> https://lcsc.com/product-detail/Voltage-Regulators-Linear-L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
