File: hardware/pcb/kicad/microcontroller.kicad_sch (KiCad schematic)
At the start: 33 parts, among them Q1 2N7002VC-, Q2 2N7002VC-, SW18 SWITCH, U1 W25Q64JV, U6 RP2040, U7 74LVC1T45, Y1 12MHz

Commit message: Reformatting, removing old files, add better documentation about licenses
Other:
- title: Mathpad -> Mathpad PCB
Changed lines of the file:
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@@
 	(paper "A4")
 	(title_block
-		(title "Mathpad")
-		(date "2025-04-05")
+		(title "Mathpad PCB")
+		(date "2025-04-07")
 		(rev "1.6")
 		(company "Summacogni OÜ")

Commit message: minor fixes
Parts:
- U1: footprint Package_SON:WSON-8-1EP_8x6mm_P1.27mm_EP3.4x4.3mm -> mathpad:WSON-8-1EP_8x6mm_P1.27mm_EP3.4x4.3mm
Changed lines of the file:
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@@
 			)
 		)
-		(property "Footprint" "Package_SON:WSON-8-1EP_8x6mm_P1.27mm_EP3.4x4.3mm"
+		(property "Footprint" "mathpad:WSON-8-1EP_8x6mm_P1.27mm_EP3.4x4.3mm"
 			(at 71.374 41.402 0)
 			(effects

Commit message: Minor modifications to the pcb
Parts:
- Q1, Q2: JLCPCB_CORRECTION 0; 0; 180 -> (none)
- U7: JLCPCB_CORRECTION 0; 0; 270 -> (none)

Commit message: Add MPN and purchase links to all components
Parts:
- C10, C11: value 1u -> 1uF X5R ±10% 25V; MPN  1uF 20% 10V 0402 -> CL05A105KA5NQNC; Purchase link (none) -> https://lcsc.com/product-detail/Multilayer-Ceramic-Capacito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
- C12, C13, C14, C15, C16, C17, C18, C19, C7: value 100n -> 100nF X7R ±10% 16V; MPN  100nF 10% 10V 0402 -> CL05B104KO5NNNC; Purchase link (none) -> https://lcsc.com/product-detail/Multilayer-Ceramic-Capacito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
- C3, C4: value 4.7u -> 4.7uF X5R ±10% 10V; MPN  4.7uF 20% 10V 0402 -> CL10A475KP8NNNC; Purchase link (none) -> https://lcsc.com/product-detail/Multilayer-Ceramic-Capacito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
- C6, C8: value 30p -> 30pF C0G ±5% 50V; Purchase link (none) -> https://lcsc.com/product-detail/Multilayer-Ceramic-Capacito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
- Q1, Q2: value 2N7002VC- -> 2N7002VC; Purchase link (none) -> https://lcsc.com/product-detail/MOSFETs_Jiangsu-Changjing-E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
- R1, R11, R2, R3: MPN  10k 1% 0402 -> 0402WGF1002TCE; Purchase link (none) -> https://lcsc.com/product-detail/Chip-Resistor-Surface-Mount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
- R12, R13: value 27 -> 27 1%; MPN  27 1% 0402 -> 0603WAF270JT5E; Purchase link (none) -> https://lcsc.com/product-detail/Chip-Resistor-Surface-Mount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
- R14, R9: value 1k -> 1k 1%; MPN  1k 1% 0402 -> 0402WGF1001TCE; Purchase link (none) -> https://lcsc.com/product-detail/Chip-Resistor-Surface-Mount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
- R4, R5, R6: value 51k -> 51k 1%; MPN  51k 1% 0402 -> 0402WGF5102TCE; Purchase link (none) -> https://lcsc.com/product-detail/Chip-Resistor-Surface-Mount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
- SW18: value SWITCH -> 1P1T; Purchase link (none) -> https://lcsc.com/product-detail/Tactile-Switches_XKB-Connec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
- U1: value W25Q64JV -> W25Q64JVZEIQ; MPN  (none) -> W25Q64JVZEIQ; Purchase link (none) -> https://lcsc.com/product-detail/NOR-FLASH_Winbond-Elec-W25Q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
- U6: MPN  SC0914(13) -> RP2040; Purchase link (none) -> https://lcsc.com/product-detail/Microcontrollers-MCU-MPU-SO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
- U7: Purchase link (none) -> https://lcsc.com/product-detail/Translators-Level-Shifters_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
- Y1: Purchase link (none) -> https://lcsc.com/product-detail/Crystals_YXC-Crystal-Oscill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
